Commit message: 修复：小车轮子离地导致无法运动

File: description/robot.xacro (robot description, xacro)
@@ -236,5 +236,5 @@
     <parent link="base_link"/>
     <child link="left_wheel_link"/>
-    <origin xyz="0 0.18 -0.04" rpy="0 0 0"/>
+    <origin xyz="0 0.18 0.025" rpy="0 0 0"/>
     <axis xyz="0 1 0"/>
   </joint>
@@ -258,5 +258,5 @@
     <parent link="base_link"/>
     <child link="right_wheel_link"/>
-    <origin xyz="0 -0.18 -0.04" rpy="0 0 0"/>
+    <origin xyz="0 -0.18 0.025" rpy="0 0 0"/>
     <axis xyz="0 -1 0"/>
   </joint>
@@ -279,5 +279,5 @@
     <parent link="base_link"/>
     <child link="caster_wheel_link"/>
-    <origin xyz="-0.2 0 -0.09" rpy="0 0 0"/>
+    <origin xyz="-0.2 0 -0.01" rpy="0 0 0"/>
   </joint>
   <!-- ========== Diff Drive Plugin ========== -->
